Commit message: update topic names and rename launch files

File: spot_driver_plus/urdf/gen3.urdf.xacro (robot description, xacro)
@@ -49,11 +49,11 @@
     sim_isaac="$(arg sim_isaac)"
     use_external_cable="$(arg use_external_cable)" >
-    <origin xyz="0.1656 0 0.12" rpy="0 0 0" />  <!-- position robot in the world -->
+    <origin xyz="0.3 0 0.085" rpy="0 0 0" />  <!-- position robot in the world -->
   </xacro:load_robot>
-  <!-- Front CB -->
-  <link name="front_collision">
+  <!-- Back CB -->
+  <link name="rear_collision">
   <visual>
     <geometry>
-    <box size="0.2 0.15 0.15" />
+    <box size="0.55 0.10 0.10" />
     </geometry>
     <material name="red">
@@ -63,26 +63,5 @@
   <collision>
     <geometry>
-    <box size="0.2 0.15 0.15" />
-    </geometry>
-  </collision>
-  </link>
-  <joint name="body_front_collision" type="fixed">
-    <child link="front_collision" />
-    <parent link="body" />
-    <origin xyz="0.3 0 0.15" rpy="0 0 0" />
-  </joint>
-  <!-- Back CB -->
-  <link name="rear_collision">
-  <visual>
-    <geometry>
-    <box size="0.6 0.14 0.14" />
-    </geometry>
-    <material name="red">
-    <color rgba="1 0 0 1" />
-    </material>
-  </visual>
-  <collision>
-    <geometry>
-    <box size="0.6 0.14 0.14" />
+    <box size="0.55 0.10 0.10" />
     </geometry>
   </collision>
@@ -91,5 +70,26 @@
     <child link="rear_collision" />
     <parent link="body" />
-    <origin xyz="-0.15 0 0.17" rpy="0 0 0" />
+    <origin xyz="-0.05 0 0.15" rpy="0 0 0" />
+  </joint>
+  <!-- Front CB -->
+  <link name="front_collision">
+    <visual>
+        <geometry>
+        <box size="0.10 0.10 0.10" />
+        </geometry>
+        <material name="red">
+        <color rgba="1 0 0 1" />
+        </material>
+    </visual>
+    <collision>
+        <geometry>
+        <box size="0.10 0.10 0.10" />
+        </geometry>
+    </collision>
+    </link>
+    <joint name="body_front_collision" type="fixed">
+        <child link="front_collision" />
+        <parent link="body" />
+        <origin xyz="0.42 0 0.125" rpy="0  0.3 0" />
   </joint>
 </robot>
